File: pcb/keyboooard.kicad_pcb (KiCad board)
At the start: 2 copper layers, 318 x 134 mm, 154 parts, among them J1 OLED_128x32, SW1 SW_Push_45deg, SW10 SW_Push_45deg, SW11 SW_Push_45deg, SW12 SW_Push_45deg, SW13 SW_Push_45deg, SW14 SW_Push_45deg, SW15 SW_Push_45deg, SW16 SW_Push_45deg, SW17 SW_Push_45deg, SW18 SW_Push_45deg, SW19 SW_Push_45deg, SW2 SW_Push_45deg, SW20 SW_Push_45deg, SW21 SW_Push_45deg, SW22 SW_Push_45deg, SW23 SW_Push_45deg, SW24 SW_Push_45deg, SW25 SW_Push_45deg, SW26 SW_Push_45deg, SW27 SW_Push_45deg, SW28 SW_Push_45deg, SW29 SW_Push_45deg, SW3 SW_Push_45deg, SW30 SW_Push_45deg, SW31 SW_Push_45deg, SW32 SW_Push_45deg, SW33 SW_Push_45deg, SW34 SW_Push_45deg, SW35 SW_Push_45deg, SW36 SW_Push_45deg, SW37 SW_Push_45deg, SW38 SW_Push_45deg, SW39 SW_Push_45deg, SW4 SW_Push_45deg, SW40 SW_Push_45deg, SW41 SW_Push_45deg, SW42 SW_Push_45deg, SW43 SW_Push_45deg, SW44 SW_Push_45deg, SW45 SW_Push_45deg, SW46 SW_Push_45deg, SW47 SW_Push_45deg, SW48 SW_Push_45deg, SW49 SW_Push_45deg, SW5 SW_Push_45deg, SW50 SW_Push_45deg, SW51 SW_Push_45deg, SW52 SW_Push_45deg, SW53 SW_Push_45deg, SW54 SW_Push_45deg, SW55 SW_Push_45deg, SW56 SW_Push_45deg, SW57 SW_Push_45deg, SW58 SW_Push_45deg, SW59 SW_Push_45deg, SW6 SW_Push_45deg, SW60 SW_Push_45deg, SW61 SW_Push_45deg, SW62 SW_Push_45deg, SW63 SW_Push_45deg, SW64 SW_Push_45deg, SW65 SW_Push_45deg, SW66 SW_Push_45deg, SW67 SW_Push_45deg, SW68 SW_Push_45deg, SW7 SW_Push_45deg, SW8 SW_Push_45deg, SW9 SW_Push_45deg, U1 RP2040_Pro_Micro

Commit message: add qmk firmware
Parts:
- added REF**: MountingHole_2.2mm_M2, MountingHole:MountingHole_2.2mm_M2, F.Cu at (65.5, 75.8)
- SW14: footprint PCM_Switch_Keyboard_Hotswap_Kailh:SW_Hotswap_Kailh_MX_2.00u -> PCM_Switch_Keyboard_Hotswap_Kailh:SW_Hotswap_Kailh_MX_1.00u
- SW15: footprint PCM_Switch_Keyboard_Hotswap_Kailh:SW_Hotswap_Kailh_MX_1.00u -> PCM_Switch_Keyboard_Hotswap_Kailh:SW_Hotswap_Kailh_MX_2.00u
- moved SW14 9.52 mm to (320.4, 103.9)
- moved SW15 9.52 mm to (349.0, 103.9)
- moved D14 9.04 mm to (329.4, 111.7)
- moved D15 9.00 mm to (358.0, 111.7)
- moved REF** 1.12 mm to (306.5, 74.8)
- moved D68 1.00 mm to (367.0, 186.0)
- moved REF** 0.24 mm to (177.5, 91.8)
- moved REF** 0.24 mm to (253.5, 91.8)
- moved REF** 0.09 mm to (253.5, 191.8)
- moved REF** 0.09 mm to (177.5, 191.8)
- moved REF** 0.09 mm to (61.5, 191.8)
- moved REF** 0.09 mm to (369.5, 191.8)
- moved D62 0.07 mm to (202.5, 187.6)
Routing:
- net COL1: track 443.0 -> 418.1 mm
- net ROW1: track 387.6 -> 374.8 mm
- net COL0: track 378.1 -> 366.3 mm
- net ROW0: track 320.1 -> 311.0 mm
- net COL13: track 376.9 -> 372.8 mm
- net COL8: track 309.7 -> 306.6 mm
- net Net-(D68-A): track 5.44 -> 3.72 mm
- net RESW2 B: track 279.0 -> 280.1 mm
- net GND: track 306.6 -> 307.5 mm
- net ROW2: track 402.9 -> 402.0 mm
